Commit message: Simulator seems to be working according to spec.  Not very useful at this time (no planning etc.) but that's ok. we're getting there.

File: src/so_arm_description/urdf/so_arm_urdf.urdf (robot description, URDF)
Before this commit: robot so_arm_urdf, 7 links, 6 joints
Links:
- added link world
Joints:
- added joint world_to_base: type fixed, parent world, child Base, origin xyz=0 0 0 rpy=0 0 0

Commit message: Ok, at this point we are seeing simulation running (and failing) in rviz, but the simulation is actually runnign in gazebo also so that is our immediate goal and we are happy with the progress at this point.  Taking a few consolidation steps to ensure that we are actually in a good place

File: src/so_arm_description/urdf/so_arm_urdf.urdf (robot description, URDF)
Before this commit: robot so_arm_urdf, 8 links, 7 joints
Joints:
- joint Elbow: limit (none) -> effort=5 velocity=2.0
- joint Jaw: limit (none) -> effort=2 velocity=1.0
- joint Pitch: limit (none) -> effort=8 velocity=1.5
- joint Rotation: limit (none) -> effort=10 velocity=1.5
- joint Wrist_Pitch: limit (none) -> effort=3 velocity=2.0
- joint Wrist_Roll: limit (none) -> effort=3 velocity=2.0
